Commit message: Actualización de nodos para utilizar filtro de Kalman

File: model/robot_core.xacro (robot description, xacro)
@@ -15,4 +15,10 @@
         <xacro:property name="ultra_y" value="0.08"/>
         <xacro:property name="ultra_z" value="0.02"/>
+        <xacro:property name="imu_x_size" value="0.025"/>
+        <xacro:property name="imu_y_size" value="0.02"/>
+        <xacro:property name="imu_z_size" value="0.01"/>
+        <xacro:property name="imu_pos_x" value="0.09"/>
+        <xacro:property name="imu_pos_y" value="0.0"/>
+        <xacro:property name="imu_pos_z" value="${imu_z_size/2}"/>
         <!-- Example link -->
         <link name="${prefix}base_link">
@@ -55,5 +61,5 @@
                     <box size="${ultra_x} ${ultra_y} ${ultra_z}"/>
                 </geometry>
-                <material name="orange"/>
+                <material name="blue"/>
             </visual>
             <collision>
@@ -138,4 +144,27 @@
             </xacro:inertial_sphere>
         </link>
+        <joint name="${prefix}base_imu_joint" type="fixed">
+            <parent link="${prefix}base_link"/>
+            <child link="${prefix}imu_link"/>
+            <origin xyz="${imu_pos_x} ${imu_pos_y} ${imu_pos_z}" rpy="0 0 0"/>
+        </joint>
+        <link name="${prefix}imu_link">
+            <visual>
+                <origin xyz="0 0 0" rpy="0 0 0"/>
+                <geometry>
+                    <box size="${imu_x_size} ${imu_y_size} ${imu_z_size}"/>
+                </geometry>
+                <material name="red"/>
+            </visual>
+            <collision>
+                <origin xyz="0 0 0" rpy="0 0 0"/>
+                <geometry>
+                    <box size="${imu_x_size} ${imu_y_size} ${imu_z_size}"/>
+                </geometry>
+            </collision>
+            <xacro:inertial_box mass="0.01" x="${imu_x_size}" y="${imu_y_size}" z="${imu_z_size}">
+                <origin xyz="0 0 0" rpy="0 0 0"/>
+            </xacro:inertial_box>
+        </link>
     </xacro:macro>
 </robot>
